File: PCB_Entrega1/PCB_Entrega1.kicad_sch (KiCad schematic)
At the start: 26 parts, among them J1 Conn_01x02_Male, J2 Conn_01x02_Male, T1 2N3904, T1_c1 2N3904, T1_paso1 BD135, T2 2N3904, T2_c1 2N3904, T2_paso1 BD136, T3 2N3906, T3_c1 2N3904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

Commit message: PCB Checkpoint 2
Parts:
- added C1: 68n, Capacitor_THT:C_Disc_D4.3mm_W1.9mm_P5.00mm, symbol Device:C
- T1_paso1: value BD135 -> 2N3906; footprint Package_TO_SOT_THT:TO-126-3_Vertical -> Package_TO_SOT_THT:TO-92_Inline
- T2_paso1: value BD136 -> TIP32C
- U1: footprint Package_SO:SOIC-8_3.9x4.9mm_P1.27mm -> Package_TO_SOT_THT:TO-92_Inline
Connections:
- net GND: now also C1.2
- net at J2.1 (Pin_1), T1_paso1.3 (B), T4.3 (C)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: now also C1.1

Commit message: Add files via upload
Parts:
- removed Disipador1: Heatsink, MountingHole:MountingHole_2.2mm_M2, symbol Mechanical:Heatsink
- T1_paso1: value 2N3906 -> 2N3904
Other:
- note added: "24/04/2025"
- note added: "Esquematico Checkpoint 2, grupo 4"
- note removed: "04/04/2025"
- note removed: "Esquematico Checkpoint 1, grupo 4"
- moved on the sheet: C1, J1, J2, Out1, R1, R1_fb1, R1_lazo1, R2, R2_fb1, R2_lazo1, R_S1, R_diodo1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
