File: PCB_checkpoint2.kicad_pcb (KiCad board)
At the start: 2 copper layers, 61.2 x 66.3 mm, 26 parts, among them J1 Conn_01x02_Male, J2 Conn_01x02_Male, T1 2N3904, T1_c1 2N3904, T1_paso1 2N3904, T2 2N3904, T2_c1 2N3904, T2_paso1 TIP32C, T3 2N3906, T3_c1 2N3904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

Commit message: PCB LDO final (esperemos)
Parts:
- moved T1_paso1 3.11 mm to (151.2, 82.7)
- moved T5_fb1 1.20 mm to (163.1, 75.6)
Connections:
- R_diodo1 pad 2: Net-(U1-K) -> Net-(T1-B)
- R_ref_c1 pad 1: Net-(T1-B) -> Net-(R_ref_c1-Pad1)
- T1_paso1 pad 2: Net-(T1_paso1-C) -> Net-(J2-Pin_1)
- T1_paso1 pad 3: Net-(J2-Pin_1) -> Net-(T1_paso1-C)
- U1 pad 1: Net-(U1-K) -> Net-(T1-B)
- U1 pad 2: Net-(T1-B) -> Net-(R_ref_c1-Pad1)
- U1 pad 3: Net-(T1-B) -> Net-(R_ref_c1-Pad1)
Routing:
- net Net-(R_ref_c1-Pad1): track 0.00 -> 7.48 mm
- net Net-(U1-K): track 7.33 -> 0.00 mm
- net Net-(T5_fb1-B): track 19.6 -> 25.6 mm
- net Net-(J1-Pin_1): track 21.1 -> 16.9 mm
- net Net-(T1-B): track 58.3 -> 61.1 mm
- net Net-(J2-Pin_1): track 86.1 -> 83.9 mm
- net Net-(T1_paso1-C): track 11.6 -> 9.58 mm
- net Net-(T1_c1-E): track 5.72 -> 3.76 mm
- net Net-(T4-E): track 4.91 -> 3.91 mm
- net Net-(T3-E): track 4.92 -> 3.92 mm
- net Net-(T1-E): track 29.4 -> 30.2 mm
Other:
- board size 61.2 x 66.3 mm -> 65 x 66.3 mm
