File: PCB_checkpoint2.kicad_sch (KiCad schematic)
At the start: 26 parts, among them J1 Conn_01x02_Male, J2 Conn_01x02_Male, T1 2N3904, T1_c1 2N3904, T1_paso1 2N3904, T2 2N3904, T2_c1 2N3904, T2_paso1 TIP32C, T3 2N3906, T3_c1 2N3904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

Commit message: PCB LDO final (esperemos)
Parts:
- removed T1_paso1: 2N3904, Package_TO_SOT_THT:TO-92_Inline, symbol Transistor_BJT:BD135
- added T1_paso1: 2N3904, Package_TO_SOT_THT:TO-92_Inline, symbol Transistor_BJT:2N3904
Connections:
- net at C1.1, J2.1 (Pin_1), T4.3 (C)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: now also T1_paso1.2 (B)
- net at R2_fb1.1, R_S1.1, T2_paso1.2 (C): now also T1_paso1.1 (E)
- net at T2_paso1.3 (B): now also T1_paso1.3 (C)
Other:
- moved on the sheet: U1
