File: PCB_checkpoint3/PCB_checkpoint3.kicad_pcb (KiCad board)
At the start: 2 copper layers, 65 x 66.3 mm, 26 parts, among them J1 Conn_01x02_Male, J2 Conn_01x02_Male, T1 2N3904, T1_c1 2N3904, T1_paso1 2N3904, T2 2N3904, T2_c1 2N3904, T2_paso1 TIP32C, T3 2N3906, T3_c1 2N3904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

Commit message: .
Parts:
- C1: value 68n -> 100n
- R1_lazo1, R2_lazo1: value 100K -> 4.7K
- moved R_S1 21.8 mm to (126.8, 88.2)
- moved C1 21.8 mm to (145.0, 70.6)
- moved J1 21.8 mm to (151.7, 119.4)
- moved J2 21.8 mm to (165.2, 119.4)
- moved Out1 21.8 mm to (169.5, 77.0)
- moved R1 21.8 mm to (151.7, 98.1)
- moved R1_fb1 21.8 mm to (155.9, 80.5)
- moved R2 21.8 mm to (165.2, 97.9)
- moved R2_fb1 21.8 mm to (142.1, 80.7)
- moved T1 21.8 mm to (154.2, 127.9)
- moved T1_c1 21.8 mm to (133.9, 127.7)
- moved T1_paso1 21.8 mm to (129.5, 81.1)
- moved T3 21.8 mm to (151.7, 110.6)
- moved T3_c1 21.8 mm to (125.6, 127.6)
- moved T4 21.8 mm to (165.2, 110.4)
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Connections:
- R_ref_c1 pad 1: Net-(R_ref_c1-Pad1) -> Net-(T1-B)
- U1 pad 2: Net-(R_ref_c1-Pad1) -> GND
- U1 pad 3: Net-(R_ref_c1-Pad1) -> GND
Routing:
- net GND: track 0.00 -> 19.8 mm
- net Net-(T1-B): track 61.1 -> 72.3 mm
- net Net-(R_ref_c1-Pad1): track 7.48 -> 0.00 mm
Other:
- board text added: "09/05/2025"
- board text added: "PCB checkpoint 3, grupo 4"
- board text removed: "24/04/2025"
- board text removed: "PCB checkpoint 2, grupo 4"
