File: PCB_checkpoint3/PCB_checkpoint3.kicad_sch (KiCad schematic)
At the start: 26 parts, among them J1 Conn_01x02_Male, J2 Conn_01x02_Male, T1 2N3904, T1_c1 2N3904, T1_paso1 2N3904, T2 2N3904, T2_c1 2N3904, T2_paso1 TIP32C, T3 2N3906, T3_c1 2N3904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

Commit message: .
Parts:
- C1: value 68n -> 100n
- R1_lazo1, R2_lazo1: value 100K -> 4.7K
Other:
- note added: "09/05/2025"
- note added: "Esquematico Checkpoint 3, grupo 4"
- note removed: "24/04/2025"
- note removed: "Esquematico Checkpoint 2, grupo 4"
Changed lines of the file:
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@@
 		)
 	)
-	(text "24/04/2025"
+	(text "09/05/2025"
 		(exclude_from_sim no)
 		(at 210.058 194.056 0)
@@
 		)
 	)
-	(text "Esquematico Checkpoint 2, grupo 4\n"
+	(text "Esquematico Checkpoint 3, grupo 4\n"
 		(exclude_from_sim no)
 		(at 187.198 190.246 0)
@@
 			)
 		)
-		(property "Value" "100K"
+		(property "Value" "4.7K"
 			(at 223.52 87.6299 0)
 			(effects
@@
 			)
 		)
-		(property "Value" "68n"
+		(property "Value" "100n"
 			(at 135.89 81.2799 0)
 			(effects
@@
 			)
 		)
-		(property "Value" "100K"
+		(property "Value" "4.7K"
 			(at 223.52 107.9499 0)
 			(effects
