File: checkpoint4/PCB_Buck/PCB_Buck.kicad_sch (KiCad schematic)
At the start: 14 parts, among them Q1 NMOS, Q2 NMOS, U1 IR2104

Commit message: PCB Buck
Connections:
- net at C1.2, U1.6 (VS): now also L1.2, Q1.3 (S), Q2.1 (D)
Changed lines of the file:
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@@
+	)
+	(junction
+		(at 120.65 102.87)
+		(diameter 0)
+		(color 0 0 0 0)
 	)
 	(junction
@@
 		)
 		(stroke
+			(width 0)
+			(type default)
+		)
+	)
+	(wire
+		(pts
+			(xy 120.65 102.87) (xy 153.67 102.87)
+		)
+		(stroke

Commit message: PCB Buck
Parts:
- removed BT2: pulso, TerminalBlock:TerminalBlock_bornier-2_P5.08mm, symbol Device:Battery_Cell
- added BT4: Battery, TerminalBlock:TerminalBlock_bornier-2_P5.08mm, symbol Device:Battery
- added C5: C, symbol Device:C
- added C6: C, Capacitor_THT:C_Disc_D4.3mm_W1.9mm_P5.00mm, symbol Device:C
- added R1, R2: R, symbol Device:R
- added R10: 1k, Resistor_THT:R_Axial_DIN0207_L6.3mm_D2.5mm_P7.62mm_Horizontal, symbol Device:R
- added R3: 100k, Resistor_THT:R_Axial_DIN0207_L6.3mm_D2.5mm_P7.62mm_Horizontal, symbol Device:R
- added R4, R9: R, Resistor_THT:R_Axial_DIN0207_L6.3mm_D2.5mm_P7.62mm_Horizontal, symbol Device:R
- added R7: 50k, Resistor_THT:R_Axial_DIN0207_L6.3mm_D2.5mm_P7.62mm_Horizontal, symbol Device:R
- added R8: 47k, Resistor_THT:R_Axial_DIN0207_L6.3mm_D2.5mm_P7.62mm_Horizontal, symbol Device:R
- added unit 2 of U1
- added unit 3 of U1
- added U2: LM393, Package_DIP:CERDIP-8_W7.62mm_SideBrazed_LongPads, symbol Comparator:LM393
- renumbered R1 to R5, R2 to R6
Connections:
- net GND: now also BT4.2 (-), C6.2, R4.2, U1.4 (V-), U2.4 (V-)
- net Salida_pwm: now reaches U1.2 (IN)
- new net: C6.1, R10.1, U2.7
- new net: R10.2, R2.2
- new net: BT4.1 (+), R2.1, R3.1, R9.1, U1.8 (V+), U2.8 (V+)
- new net: R7.1, R8.1, U2.3 (+)
- new net: R1.1, R7.2, R9.2, U2.1
- new net: C5.2, R8.2, U2.1, U2.6 (-)
- new net: C5.1, R1.2, U2.2 (-)
- new net: U1.6 (-), U1.7, U2.2 (-), U2.3 (+)
- new net: R3.2, R4.1, U1.5 (+)
- new net VREF: U2.5 (+)
Other:
- moved on the sheet: BT1, BT3, C1, C2, C3, C4, D1, L1, Q1, Q2, R5, R6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
