File: checkpoint5/pcb_final.kicad_pcb (KiCad board)
At the start: 2 copper layers, 42 parts, among them J1 Conn_01x02_Pin, Q1 NMOS, Q2 NMOS, U1 TL072, U2 LM393, U3 IR2104, U4 TL072, U5 LM317L_SOT-89, U6 TL431LP

Commit message: Add files via upload
Parts:
- moved R5 4.81 mm to (163.2, 80.2)
- moved BT1 4.49 mm to (168.0, 111.0)
- moved Ccami1 2.92 mm to (166.8, 98.2)
- moved U5 1.05 mm to (169.2, 85.8), turned to 180 degrees
- moved r_i1 0.12 mm to (101.3, 100.1)
- turned R7 to 90 degrees
Routing:
- net Vin: track 37.2 -> 45.0 mm
- net Net-(D2-A): track 71.5 -> 76.7 mm
- net Net-(U5-ADJ): track 9.42 -> 13.2 mm
