File: checkpoint5/pcb_cp5_cami/pcb_check4_pwm.kicad_pcb (KiCad board)
At the start: 2 copper layers, 42 parts, among them J1 Conn_01x02_Pin, Q1 NMOS, Q2 NMOS, U1 TL072, U2 LM393, U3 IR2104, U4 TL072, U5 LM317L_SOT-89, U6 TL431LP

Commit message: Add files via upload
Parts:
- removed the C1 at (112.5, 96.8)
- removed the C2 at (86.9, 79.2)
- added C7: C, Capacitor_THT:C_Axial_L5.1mm_D3.1mm_P7.50mm_Horizontal, F.Cu at (92.8, 79.0)
- added C8: C, Capacitor_THT:C_Axial_L5.1mm_D3.1mm_P7.50mm_Horizontal, F.Cu at (107.0, 97.0)
- added J2: Conn_01x01, Connector_PinHeader_1.27mm:PinHeader_1x01_P1.27mm_Vertical, F.Cu at (140.6, 83.6)
- added J3: Conn_01x02, Connector_PinHeader_1.27mm:PinHeader_1x02_P1.27mm_Vertical, F.Cu at (144.4, 81.2)
- moved Ccami1 46.1 mm to (165.1, 80.5)
- moved D2 31.8 mm to (169.8, 90.7), turned to -90 degrees
- moved R9 24.5 mm to (162.3, 87.0), turned to 180 degrees
- moved R10 21.0 mm to (150.4, 101.2), turned to 0 degrees
- moved BT1 19.2 mm to (152.2, 107.2)
- moved U5 16.7 mm to (131.5, 107.9), turned to 0 degrees
- moved D3 16.1 mm to (183.8, 106.0), turned to 0 degrees
- moved D1 16.1 mm to (144.2, 87.2), turned to 180 degrees
- moved Q1 14.7 mm to (161.2, 92.0), turned to -90 degrees
- moved U3 12.7 mm to (139.2, 92.4)
- moved C1 9.20 mm to (151.0, 90.0)
- moved R5 8.30 mm to (129.3, 97.0), turned to 180 degrees
- moved L1 6.50 mm to (179.2, 89.5)
- moved Q2 4.44 mm to (165.0, 103.5), turned to 0 degrees
- moved R7 3.00 mm to (129.3, 100.8)
Connections:
- C5 pad 1: Vref -> Net-(J3-Pin_2)
- C6 pad 1: Vref -> Net-(J3-Pin_2)
- U4 pad 1: Vref -> Net-(J3-Pin_2)
Routing:
- net Net-(J3-Pin_2): track 0.00 -> 15.5 mm
- net Net-(D1-K): track 26.3 -> 15.9 mm
- net Vin: track 45.7 -> 56.1 mm
- net Net-(U3-VS): track 13.3 -> 4.20 mm
- net Net-(D2-A): track 39.1 -> 48.1 mm
- net Net-(U3-LO): track 12.7 -> 4.12 mm
- net Net-(J1-Pin_1): track 42.1 -> 35.7 mm
- net Net-(J2-Pin_1): track 52.1 -> 56.4 mm
- net Vref: track 37.5 -> 33.8 mm
- net Net-(Q2-G): track 4.85 -> 7.84 mm
- net Net-(U5-ADJ): track 13.6 -> 16.6 mm
- net Net-(Q1-G): track 5.92 -> 4.92 mm
