File: checkpoint5/pcb_cp5_cami/pcb_check4_pwm.kicad_sch (KiCad schematic)
At the start: 40 parts, among them J1 Conn_01x02_Pin, Q1 NMOS, Q2 NMOS, U1 TL072, U2 LM393, U3 IR2104, U4 TL072, U5 LM317L_SOT-89, U6 TL431LP

Commit message: Add files via upload
Parts:
- added C7, C8: C, Capacitor_THT:C_Axial_L5.1mm_D3.1mm_P7.50mm_Horizontal, symbol Device:C
- added J2: Conn_01x01, Connector_PinHeader_1.27mm:PinHeader_1x01_P1.27mm_Vertical, symbol Connector_Generic:Conn_01x01
- added J3: Conn_01x02, Connector_PinHeader_1.27mm:PinHeader_1x02_P1.27mm_Vertical, symbol Connector_Generic:Conn_01x02
Connections:
- net GND: now also C7.2, C8.2
- net Vref: now also J3.1 (Pin_1); no longer C5.1, C6.1, U4.1
- net Vreg: now also C7.1, C8.1
- net at R6.1, U2.7, U3.2 (IN): now also J2.1 (Pin_1)
- new net: C5.1, C6.1, J3.2 (Pin_2), U4.1
